Commit message: added navigation folder

File: src/diff_drive_description/urdf/diff_drive.xacro (robot description, xacro)
@@ -12,30 +12,29 @@
     />
     <xacro:mechanical
-    base_ln_xyz="-0.412 -0.14 -0.086"
+    base_ln_xyz="0 0 0"
     base_ln_rpy="0 0 0"
-    base_ln_mass="0.1"
+    base_ln_mass="2.5"
     wheel_l_ln="left_wheel"
     wheel_r_ln="right_wheel"
-    wheel_l_xyz="-0.155 -0.04 0.08"
-    wheel_r_xyz="0.135 -0.04 0.08"
-    wheel_l_rpy="0 1.54 0"
-    wheel_r_rpy="0 1.54 0"
-    wheel_mass="0.08"
-    wheel_rad="0.08"
+    wheel_l_xyz="-0.1 0.145 0.04"
+    wheel_r_xyz="-0.1 -0.145 0.04"
+    wheel_l_rpy="0 0 0"
+    wheel_r_rpy="0 0 0"
+    wheel_mass="0.2"
+    wheel_rad="0.04"
     caster_ln="caster"
-    caster_xyz="-0.015 0.25 0"
-    caster_rpy="1.54 0 1.54"
-    caster_mass="0.05"
+    caster_xyz="0.156 0 0.034"
+    caster_rpy="0 0 0"
+    caster_mass="0.4"
     lidar_ln="rplidar"
-    lidar_xyz="0 0 0.04"
+    lidar_xyz="0.16 0 0.155"
     lidar_rpy="0 0 0"
-    lidar_mass="0.03"
+    lidar_mass="0.1"
     camera_ln="camera"
-    camera_xyz="0.05 0 0.04"
+    camera_xyz="0.205 -0.0005 0.105"
     camera_rpy="0 0 0"
-    camera_mass="0.03"
-    camera_name="camera"
+    camera_mass="0.1"
     imu_ln="imu"
-    imu_xyz="-0.04 0 0.04"
+    imu_xyz="-0.05 0 0.07"
     imu_rpy="0 0 0"
     imu_mass="0.01"

File: src/diff_drive_description/urdf/gazebo.xacro (robot description, xacro)
@@ -6,18 +6,20 @@
     <gazebo>
         <plugin name="differential_drive_controller" filename="libgazebo_ros_diff_drive.so">
+          <alwaysOn>true</alwaysOn>
           <!-- Plugin update rate in Hz -->
           <updateRate>20</updateRate>
           <!-- Name of left joint, defaults to `left_joint` -->
-          <leftJoint>{wheel_l_ln}_joint</leftJoint>
+          <leftJoint>${wheel_l_ln}_joint</leftJoint>
           <!-- Name of right joint, defaults to `right_joint` -->
-          <rightJoint>{wheel_r_ln}_joint</rightJoint>
+          <rightJoint>${wheel_r_ln}_joint</rightJoint>
           <!-- The distance from the center of one wheel to the other, in meters, defaults to 0.34 m -->
-          <wheelSeparation>0.5380</wheelSeparation>
+          <wheelSeparation>0.29</wheelSeparation>
           <!-- Diameter of the wheels, in meters, defaults to 0.15 m -->
-          <wheelDiameter>0.8</wheelDiameter>
+          <wheelDiameter>0.08</wheelDiameter>
           <!-- Wheel acceleration, in rad/s^2, defaults to 0.0 rad/s^2 -->
-          <wheelAcceleration>1.0</wheelAcceleration>
-          <!-- Maximum torque which the wheels can produce, in Nm, defaults to 5 Nm -->
-          <wheelTorque>20</wheelTorque>
+          <wheelAcceleration>0</wheelAcceleration>
+          <!-- Maximum torque which the wheels can produce, in Nm, defaults to 5 Nm-->
+          <wheelTorque>5</wheelTorque>
+          <torque>5</torque>
           <!-- Topic to receive geometry_msgs/Twist message commands, defaults to `cmd_vel` -->
           <commandTopic>cmd_vel</commandTopic>
@@ -29,37 +31,39 @@
           <robotBaseFrame>base_footprint</robotBaseFrame>
           <!-- Odometry source, 0 for ENCODER, 1 for WORLD, defaults to WORLD -->
-          <odometrySource>1</odometrySource>
+          <odometrySource>world</odometrySource>
           <!-- Set to true to publish transforms for the wheel links, defaults to false -->
           <publishWheelTF>false</publishWheelTF>
           <!-- Set to true to publish transforms for the odometry, defaults to true -->
-          <publishOdom>true</publishOdom>
+          <!-- <publishOdom>true</publishOdom> -->
           <!-- Set to true to publish sensor_msgs/JointState on /joint_states for the wheel joints, defaults to false -->
-          <publishWheelJointState>true</publishWheelJointState>
+          <publishWheelJointState>false</publishWheelJointState>
           <!-- Set to true to swap right and left wheels, defaults to true -->
           <legacyMode>false</legacyMode>
           <!-- Set to true to publish transforms, defaults to true -->
-          <publishTf>true</publishTf>
+          <publishOdomTF>true</publishOdomTF>
+          <publishTf>1</publishTf>
+          <rosDebugLevel>na</rosDebugLevel>
         </plugin>
     </gazebo>
-    <gazebo reference="${camera_ln_n}">
-        <sensor name="${camera_ln_n}_camera" type="depth">
+    <gazebo reference="${camera_ln_n}_link">
+        <sensor name="${camera_ln_n}" type="depth">
           <update_rate>20</update_rate>
           <camera>
-            <horizontal_fov>1.047198</horizontal_fov>
+            <horizontal_fov>1.1</horizontal_fov>
             <image>
-              <width>640</width>
-              <height>480</height>
+              <width>720</width>
+              <height>640</height>
               <format>R8G8B8</format>
             </image>
             <clip>
-              <near>0.05</near>
-              <far>3</far>
+              <near>0.1</near>
+              <far>8.0</far>
             </clip>
           </camera>
           <plugin name="${camera_ln_n}_controller" filename="libgazebo_ros_openni_kinect.so">
-            <baseline>0.2</baseline>
+            <baseline>0.1</baseline>
             <alwaysOn>true</alwaysOn>
-            <updateRate>1.0</updateRate>
-            <cameraName>${camera_name}_ir</cameraName>
+            <updateRate>20</updateRate>
+            <cameraName>${camera_name}</cameraName>
             <imageTopicName>/${camera_name}/color/image_raw</imageTopicName>
             <cameraInfoTopicName>/${camera_name}/color/camera_info</cameraInfoTopicName>
@@ -67,25 +71,20 @@
             <depthImageInfoTopicName>/${camera_name}/depth/camera_info</depthImageInfoTopicName>
             <pointCloudTopicName>/${camera_name}/depth/points</pointCloudTopicName>
-            <frameName>${camera_ln_n}_link</frameName>
-            <pointCloudCutoff>0.5</pointCloudCutoff>
-            <pointCloudCutoffMax>3.0</pointCloudCutoffMax>
-            <distortionK1>0.00000001</distortionK1>
-            <distortionK2>0.00000001</distortionK2>
-            <distortionK3>0.00000001</distortionK3>
-            <distortionT1>0.00000001</distortionT1>
-            <distortionT2>0.00000001</distortionT2>
-            <CxPrime>0</CxPrime>
-            <Cx>0</Cx>
-            <Cy>0</Cy>
-            <focalLength>0</focalLength>
-            <hackBaseline>0</hackBaseline>
+            <frameName>${camera_ln_n}_frame</frameName>
+            <pointCloudCutoff>0.1</pointCloudCutoff>
+            <pointCloudCutoffMax>8.0</pointCloudCutoffMax>
+            <distortion_k1>0.0</distortion_k1>
+            <distortion_k2>0.0</distortion_k2>
+            <distortion_k3>0.0</distortion_k3>
+            <distortion_t1>0.0</distortion_t1>
+            <distortion_t2>0.0</distortion_t2>
           </plugin>
         </sensor>
     </gazebo>
-    <gazebo reference="${imu_ln_n}">
+    <gazebo reference="${imu_ln_n}_link">
         <gravity>true</gravity>
-        <sensor name="imu_sensor" type="imu">
+        <sensor name="${imu_ln_n}_link" type="imu">
           <always_on>true</always_on>
-          <update_rate>100</update_rate>
+          <update_rate>20</update_rate>
           <visualize>true</visualize>
           <topic>__default_topic__</topic>
@@ -103,4 +102,54 @@
         </sensor>
     </gazebo>
+    <gazebo reference="${lidar_ln}_link">
+       <sensor type="ray" name="head_rplidar_sensor">
+         <pose>0 0 0 0 0 0</pose>
+         <visualize>false</visualize>
+         <update_rate>100</update_rate>
+         <ray>
+           <scan>
+             <horizontal>
+               <samples>1920</samples>
+               <resolution>1</resolution>
+               <min_angle>-3.14159265</min_angle>
+               <max_angle>3.14159265</max_angle>
+             </horizontal>
+           </scan>
+           <range>
+             <min>0.2</min>
+             <max>12.0</max>
+             <resolution>1.0</resolution>
+           </range>
+           <noise>
+             <type>gaussian</type>
+             <mean>0.0</mean>
+             <stddev>0.01</stddev>
+           </noise>
+         </ray>
+         <plugin name="gazebo_ros_head_rplidar_controller" filename="libgazebo_ros_laser.so">
+           <topicName>/scan</topicName>
+           <robotNamespace>/laser_scan/scan</robotNamespace>
+           <frameName>rplidar_link</frameName>
+         </plugin>
+       </sensor>
+     </gazebo>
+    <gazebo reference="base_frame">
+      <material>Gazebo/Gold</material>
+    </gazebo>
+    <gazebo reference="${wheel_r_ln}_link">
+      <material>Gazebo/Red</material>
+    </gazebo>
+    <gazebo reference="${wheel_l_ln}_link">
+      <material>Gazebo/Red</material>
+    </gazebo>
+    <gazebo reference="${imu_ln_n}_link">
+      <material>Gazebo/Black</material>
+    </gazebo>
+    <gazebo reference="${camera_ln_n}_link">
+      <material>Gazebo/White</material>
+    </gazebo>
+    <gazebo reference="${lidar_ln}_link">
+      <material>Gazebo/Black</material>
+    </gazebo>
     </xacro:macro>
 </robot>

File: src/diff_drive_description/urdf/mechanical.xacro (robot description, xacro)
@@ -2,60 +2,24 @@
 <robot xmlns:xacro="http://www.ros.org/wiki/xacro">
     <!-- Sensor models -->
-	<!-- <xacro:include filename="$(find diff_drive_description)/urdf/sensor.xacro" /> -->
-    <material name="Black">
-        <color rgba="0.0 0.0 0.0 1.0"/>
-    </material>
-    <material name="Red">
-        <color rgba="0.8 0.0 0.0 1.0"/>
-    </material>
-    <material name="White">
-        <color rgba="1.0 1.0 1.0 1.0"/>
-    </material>
-    <material name="Green">
-        <color rgba="0.0 0.8 0.0 1.0"/>
-    </material>
-	<xacro:macro name="cylinder_inertia" params="m r h">
-        <inertia
-            ixx="${m*(3*r*r+h*h)/12}"
-                    ixy = "0"
-                    ixz = "0"
-                    iyy="${m*(3*r*r+h*h)/12}"
-                    iyz = "0"
-                    izz="${m*r*r/2}"
-        />
-    </xacro:macro>
-    <xacro:macro name="box_inertia" params="m l w h">
-        <inertia
-            ixx="${m*(w*w+h*h)/12}"
-                    ixy = "0"
-                    ixz = "0"
-                    iyy="${m*(l*l+h*h)/12}"
-                    iyz = "0"
-                    izz="${m*(l*l+h*h)/12}"
-        />
-    </xacro:macro>
+	<xacro:include filename="$(find diff_drive_description)/urdf/sensor.xacro" />
     <xacro:macro
     name="mechanical"
-    params="base_ln_xyz base_ln_rpy base_ln_mass wheel_l_ln wheel_r_ln wheel_l_xyz wheel_r_xyz wheel_l_rpy wheel_r_rpy wheel_mass wheel_rad caster_ln caster_xyz caster_rpy caster_mass lidar_ln lidar_xyz lidar_rpy lidar_mass camera_ln camera_xyz camera_rpy camera_mass camera_name imu_ln imu_xyz imu_rpy imu_mass" >
+    params="base_ln_xyz base_ln_rpy base_ln_mass wheel_l_ln wheel_r_ln wheel_l_xyz wheel_r_xyz wheel_l_rpy wheel_r_rpy wheel_mass wheel_rad caster_ln caster_xyz caster_rpy caster_mass lidar_ln lidar_xyz lidar_rpy lidar_mass camera_ln camera_xyz camera_rpy camera_mass imu_ln imu_xyz imu_rpy imu_mass" >
 	<link name="base_footprint"/>
-	<link name='base_link'>
+	<link name='base_frame'>
 		<collision>
-			<origin xyz="${base_ln_xyz}"
-					rpy="${base_ln_rpy}"/>
 			<geometry>
-				<mesh filename="package://diff_drive_description/meshes/main.STL" scale="0.001 0.001 0.001"/>
+				<mesh filename="package://diff_drive_description/meshes/main.STL" scale="1 1 1"/>
 			</geometry>
 		</collision>
 		<visual>
-			<origin xyz="${base_ln_xyz}"
-					rpy="${base_ln_rpy}"/>
 			<geometry>
-				<mesh filename="package://diff_drive_description/meshes/main.STL" scale="0.001 0.001 0.001"/>
+				<mesh filename="package://diff_drive_description/meshes/main.STL" scale="1 1 1"/>
 			</geometry>
-			<material name="White"/>
+			<material name="Gold"/>
 		</visual>
 		<inertial>
-			<origin xyz="${base_ln_xyz}"
-					rpy="${base_ln_rpy}"/>
+			<origin xyz="-0.1 0 0.1"
+					rpy="0.01 0.01 1.54"/>
 			<mass value="${base_ln_mass}"/>
 			<xacro:box_inertia
@@ -68,26 +32,22 @@
     <link name='${wheel_l_ln}_link'>
 		<collision>
-			<origin xyz="${wheel_l_xyz}"
-					rpy="${wheel_l_rpy}"/>
 			<geometry>
-				<mesh filename="package://diff_drive_description/meshes/wheel_80mm.STL" scale="0.001 0.01 0.001"/>
+				<mesh filename="package://diff_drive_description/meshes/wheel_80mm.STL" scale="1 1 1"/>
 			</geometry>
 		</collision>
 		<visual>
-			<origin xyz="${wheel_l_xyz}"
-					rpy="${wheel_l_rpy}"/>
 			<geometry>
-				<mesh filename="package://diff_drive_description/meshes/wheel_80mm.STL" scale="0.001 0.001 0.001"/>
+				<mesh filename="package://diff_drive_description/meshes/wheel_80mm.STL" scale="1 1 1"/>
 			</geometry>
-			<material name="Green"/>
+			<material name="Red"/>
 		</visual>
 		<inertial>
-			<origin xyz="${wheel_l_xyz}"
-					rpy="${wheel_l_rpy}"/>
+			<origin xyz="0 0 0"
+					rpy="1.54 0 0"/>
 			<mass value="${wheel_mass}"/>
 			<xacro:cylinder_inertia
 				m="${wheel_mass}"
                 r="${wheel_rad}"
-                h="0.05"
+                h="0.015"
             />
 		</inertial>
@@ -95,26 +55,22 @@
     <link name='${wheel_r_ln}_link'>
 		<collision>
-			<origin xyz="${wheel_r_xyz}"
-					rpy="${wheel_r_rpy}"/>
 			<geometry>
-				<mesh filename="package://diff_drive_description/meshes/wheel_80mm.STL" scale="0.001 0.001 0.001"/>
+				<mesh filename="package://diff_drive_description/meshes/wheel_80mm.STL" scale="1 1 1"/>
 			</geometry>
 		</collision>
 		<visual>
-			<origin xyz="${wheel_r_xyz}"
-					rpy="${wheel_r_rpy}"/>
 			<geometry>
-				<mesh filename="package://diff_drive_description/meshes/wheel_80mm.STL" scale="0.001 0.001 0.001"/>
+				<mesh filename="package://diff_drive_description/meshes/wheel_80mm.STL" scale="1 1 1"/>
 			</geometry>
 			<material name="Red"/>
 		</visual>
 		<inertial>
-			<origin xyz="${wheel_r_xyz}"
-					rpy="${wheel_r_rpy}"/>
+			<origin xyz="0 0 0"
+					rpy="1.54 0 0"/>
 			<mass value="${wheel_mass}"/>
 			<xacro:cylinder_inertia
 				m="${wheel_mass}"
                 r="${wheel_rad}"
-                h="0.05"
+                h="0.015"
             />
 		</inertial>
@@ -122,15 +78,11 @@
 	<link name="${caster_ln}_link">
 		<collision>
-			<origin xyz="${caster_xyz}"
-					rpy="${caster_rpy}"/>
 			<geometry>
-				<mesh filename="package://diff_drive_description/meshes/caster.STL" scale="0.001 0.001 0.001"/>
+				<mesh filename="package://diff_drive_description/meshes/caster.STL" scale="1 1 1"/>
 	  		</geometry>
 		</collision>
 		<visual>
-			<origin xyz="${caster_xyz}"
-					rpy="${caster_rpy}"/>
 			<geometry>
-				<mesh filename="package://diff_drive_description/meshes/caster.STL" scale="0.001 0.001 0.001"/>
+				<mesh filename="package://diff_drive_description/meshes/caster.STL" scale="1 1 1"/>
 			</geometry>
 			<material name="Black" />
@@ -142,7 +94,7 @@
 			<xacro:box_inertia
 				m="${caster_mass}"
-				l="0.04"
-				w="0.04"
-				h="0.04"/>
+				l="0.02"
+				w="0.02"
+				h="0.02"/>
 		</inertial>
 	</link>
@@ -150,14 +102,14 @@
 		<collision>
 			<origin xyz="0 0 0"
-					rpy="0 1.54 0"/>
+					rpy="0 0 0"/>
 			<geometry>
-				<mesh filename="package://diff_drive_description/meshes/caster_wheel.stl" scale="0.02 0.02 0.02"/>
-	  		</geometry>
+				<mesh filename="package://diff_drive_description/meshes/caster_wheel.stl" scale="1 1 1"/>
+				</geometry>
 		</collision>
 		<visual>
-			<origin xyz="0 0.268 0.02"
-					rpy="0 1.54 0"/>
+			<origin xyz="0 0 0"
+					rpy="0 0 0"/>
 			<geometry>
-				<mesh filename="package://diff_drive_description/meshes/caster_wheel.stl" scale="0.025 0.025 0.025"/>
+				<mesh filename="package://diff_drive_description/meshes/caster_wheel.stl" scale="1 1 1"/>
 			</geometry>
 			<material name="White" />
@@ -166,7 +118,7 @@
 			<origin xyz="0 0 0"
 					rpy="0 0 0"/>
-			<mass value="0.02"/>
+			<mass value="0.4"/>
 			<xacro:box_inertia
-				m="0.02"
+				m="0.04"
 				l="0.04"
 				w="0.04"
@@ -176,22 +128,43 @@
     <joint name="base_joint" type="fixed">
 		<parent link="base_footprint"/>
-		<child link="base_link"/>
+		<child link="base_frame"/>
+		<origin xyz="${base_ln_xyz}" rpy="${base_ln_rpy}"/>
 	</joint>
     <joint name="${wheel_l_ln}_joint" type="continuous">
-		<parent link="base_link"/>
+		<parent link="base_frame"/>
 		<child link="${wheel_l_ln}_link"/>
+		<origin xyz="${wheel_l_xyz}" rpy="${wheel_l_rpy}"/>
+		<axis xyz="0.0 1.0 0.0"/>
 	</joint>
     <joint name="${wheel_r_ln}_joint" type="continuous">
-		<parent link="base_link"/>
+		<parent link="base_frame"/>
 		<child link="${wheel_r_ln}_link"/>
+		<origin xyz="${wheel_r_xyz}" rpy="${wheel_r_rpy}"/>
+		<axis xyz="0.0 1.0 0.0"/>
 	</joint>
     <joint name="${caster_ln}_joint" type="fixed">
-		<parent link="base_link"/>
+		<parent link="base_frame"/>
 		<child link="${caster_ln}_link"/>
+		<origin xyz="${caster_xyz}" rpy="${caster_rpy}"/>
 	</joint>
-	<joint name="caster_wheel_joint" type="fixed">
-		<parent link="base_link"/>
+	<joint name="caster_wheel_joint" type="continuous">
+		<parent link="${caster_ln}_link"/>
 		<child link="caster_wheel_link"/>
+		<origin xyz="0.0 0 -0.014" rpy="0 0 1.54"/>
 	</joint>
+	<xacro:sensor
+	lidar_ln="${lidar_ln}"
+    lidar_xyz="${lidar_xyz}"
+    lidar_rpy="${lidar_rpy}"
+    lidar_mass="${lidar_mass}"
+    camera_ln="${camera_ln}"
+    camera_xyz="${camera_xyz}"
+    camera_rpy="${camera_rpy}"
+    camera_mass="${camera_mass}"
+    imu_ln="${imu_ln}"
+    imu_xyz="${imu_xyz}"
+    imu_rpy="${imu_rpy}"
+    imu_mass="${imu_mass}"
+    />
 </xacro:macro>
 </robot>
